File: Keyboard PCB.sch (KiCad schematic (older format))
At the start: 150 parts, among them SW1 SW_Push, U1 ATmega32U4-AU, Y1 16MHz

Commit message: PCB design
Connections:
- net ROW0: now also D55.1 (K), D59.1 (K), D63.1 (K)
Changed lines of the file:
@@
 Wire Wire Line
 	9450 3200 9050 3200
+Wire Wire Line
+	10250 2000 9850 2000
+Wire Wire Line
+	9850 2000 9850 1950
+Wire Wire Line
+	9850 1950 9450 1950
+Wire Wire Line
+	9050 1950 9050 2000
+Connection ~ 9850 1950
+Connection ~ 9450 1950
+Wire Wire Line
+	9450 1950 9050 1950
+Connection ~ 9050 2000
 $EndSCHEMATC

Commit message: column traces
Parts:
- U1: footprint Housings_QFP:LQFP-64_14x14mm_Pitch0.8mm -> Package_QFP:TQFP-44_10x10mm_P0.8mm
Changed lines of the file:
@@
 F 0 "U1" H 2500 3311 50  0000 C CNN
 F 1 "ATmega32U4-AU" H 2500 3220 50  0000 C CNN
-F 2 "Housings_QFP:LQFP-64_14x14mm_Pitch0.8mm" H 2500 5200 50  0001 C CIN
+F 2 "Package_QFP:TQFP-44_10x10mm_P0.8mm" H 2500 5200 50  0001 C CIN
 F 3 "http://ww1.microchip.com/downloads/en/DeviceDoc/Atmel-7766-8-bit-AVR-ATmega16U4-32U4_Datasheet.pdf" H 2500 5200 50  0001 C CNN
 	1    2500 5200
