File: Keyboard PCB.kicad_pcb (KiCad board)
At the start: 2 copper layers, 150 parts, among them SW1 SW_Push, U1 ATmega32U4-AU, Y1 16MHz

Commit message: yes
Parts:
- C1, C2, C3, C4, C7, F1, R1, R2, R3, R4, SW1, USB1: moved to B.Cu
- U1: footprint Housings_QFP:LQFP-64_14x14mm_Pitch0.8mm -> Package_QFP:TQFP-44_10x10mm_P0.8mm
- moved USB1 210.4 mm to (34.3, -122.7), turned to 270 degrees
- moved F1 187.7 mm to (39.1, -111.5), turned to 180 degrees
- moved C3 111.1 mm to (181.2, -45.0)
- moved C4 107.7 mm to (163.8, -41.8), turned to 270 degrees
- moved R1 107.5 mm to (36.2, -103.8), turned to 90 degrees
- moved SW1 106.6 mm to (191.7, -41.5), turned to 270 degrees
- moved C1 99.4 mm to (177.5, -28.4)
- moved R2 95.5 mm to (39.5, -103.8), turned to 90 degrees
- moved C7 88.2 mm to (172.3, -46.0), turned to 180 degrees
- moved C5 79.6 mm to (184.3, -32.3), turned to 0 degrees
- moved Y1 77.9 mm to (184.2, -36.7), turned to 90 degrees
- moved C6 77.5 mm to (184.1, -41.2), turned to 180 degrees
- moved C2 68.4 mm to (163.8, -32.0), turned to 90 degrees
- moved R3 64.3 mm to (181.2, -47.5)
- moved R4 60.4 mm to (168.9, -27.9), turned to 180 degrees
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Routing:
- net ROW0: track 0.00 -> 309.3 mm
- net ROW1: track 0.00 -> 300.4 mm
- net ROW3: track 0.00 -> 297.0 mm
- net ROW2: track 0.00 -> 297.0 mm
- net ROW4: track 0.00 -> 296.8 mm, vias 0 -> 2
- net GND: track 0.00 -> 279.9 mm, vias 0 -> 8
- net +5V: track 0.00 -> 244.2 mm, vias 0 -> 8
- net Net-(R2-Pad1): track 0.00 -> 240.6 mm, vias 0 -> 2
- net Net-(R1-Pad1): track 0.00 -> 233.9 mm
- net COL12: track 0.00 -> 93.2 mm
- net COL1: track 0.00 -> 91.9 mm
- net COL2: track 0.00 -> 88.2 mm
- net COL14: track 0.00 -> 87.2 mm
- net COL5: track 0.00 -> 86.1 mm
- net COL10: track 0.00 -> 86.1 mm
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Other:
- net class Default: trace_width 0.25 -> 0.254
- net class Power added: clearance 0.2, trace_width 0.381, via_dia 0.8, via_drill 0.4

Commit message: column traces
Parts:
- moved R4 62.0 mm to (107.1, -33.1), turned to 270 degrees
- moved C3 60.1 mm to (123.7, -27.6), turned to 90 degrees
- moved SW1 58.5 mm to (133.3, -42.1)
- moved R3 57.1 mm to (124.2, -44.3), turned to 90 degrees
- moved U1 56.6 mm to (116.1, -37.7)
- moved Y1 56.6 mm to (127.6, -37.4)
- moved C5 56.6 mm to (127.7, -33.0)
- moved C6 56.6 mm to (127.5, -41.9)
- moved C7 56.5 mm to (115.9, -46.8), turned to 90 degrees
- moved C1 49.1 mm to (128.4, -27.6), turned to 90 degrees
- moved C4 44.9 mm to (121.2, -27.6), turned to 90 degrees
- moved C2 37.9 mm to (126.1, -27.6)
- moved F1 8.98 mm to (46.9, -107.2)
Connections:
- U1 pad 20: Net-(U1-Pad20) -> COL12
- U1 pad 21: Net-(U1-Pad21) -> COL13
- U1 pad 22: Net-(U1-Pad22) -> COL14
- U1 pad 37: Net-(U1-Pad37) -> ROW4
- U1 pad 38: Net-(U1-Pad38) -> ROW3
- U1 pad 39: Net-(U1-Pad39) -> ROW2
- U1 pad 40: Net-(U1-Pad40) -> ROW1
- U1 pad 41: Net-(U1-Pad41) -> ROW0
Routing:
- net Net-(R2-Pad1): track 240.6 -> 0.58 mm, vias 2 -> 0
- net Net-(R1-Pad1): track 233.9 -> 0.70 mm
- net GND: track 279.9 -> 81.3 mm, vias 8 -> 6
- net COL14: track 87.2 -> 285.3 mm, vias 0 -> 1
- net +5V: track 244.2 -> 53.4 mm, vias 8 -> 0
- net COL13: track 85.1 -> 262.0 mm, vias 0 -> 1
- net COL12: track 93.2 -> 249.2 mm, vias 0 -> 1
- net ROW0: track 309.3 -> 394.5 mm, vias 0 -> 8
- net ROW1: track 300.4 -> 363.5 mm, vias 0 -> 4
- net ROW2: track 297.0 -> 341.0 mm, vias 0 -> 2
- net ROW3: track 297.0 -> 322.8 mm
- net D+: track 16.8 -> 0.11 mm, vias 2 -> 0
- net D-: track 15.0 -> 0.00 mm, vias 2 -> 0
- net VCC: track 11.1 -> 0.00 mm, vias 2 -> 0
- net ROW4: track 296.8 -> 305.0 mm
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
Commit message: 1st routing completion
Parts:
- moved F1 6.83 mm to (42.3, -102.1), turned to 90 degrees
Connections:
- U1 pad 10: Net-(U1-Pad10) -> COL10
- U1 pad 11: Net-(U1-Pad11) -> COL11
- U1 pad 25: Net-(U1-Pad25) -> COL7
- U1 pad 26: Net-(U1-Pad26) -> COL6
- U1 pad 27: Net-(U1-Pad27) -> COL5
- U1 pad 28: Net-(U1-Pad28) -> COL4
- U1 pad 29: Net-(U1-Pad29) -> COL3
- U1 pad 30: Net-(U1-Pad30) -> COL2
- U1 pad 31: Net-(U1-Pad31) -> COL1
- U1 pad 32: Net-(U1-Pad32) -> COL0
- U1 pad 8: Net-(U1-Pad8) -> COL8
- U1 pad 9: Net-(U1-Pad9) -> COL9
Routing:
- net GND: track 81.3 -> 269.7 mm
- net COL11: track 70.0 -> 221.7 mm, vias 0 -> 1
- net Net-(R1-Pad1): track 0.70 -> 142.6 mm, vias 0 -> 2
- net COL10: track 86.1 -> 210.7 mm, vias 0 -> 1
- net Net-(R2-Pad1): track 0.58 -> 124.8 mm, vias 0 -> 2
- net +5V: track 53.4 -> 161.5 mm, vias 0 -> 6
- net COL9: track 85.1 -> 192.0 mm, vias 0 -> 1
- net COL0: track 83.6 -> 184.0 mm, vias 0 -> 1
- net COL8: track 67.0 -> 155.3 mm, vias 0 -> 1
- net COL7: track 66.1 -> 142.3 mm, vias 0 -> 1
- net COL1: track 91.9 -> 167.8 mm, vias 0 -> 1
- net COL6: track 65.2 -> 126.3 mm, vias 0 -> 1
- net COL2: track 88.2 -> 140.0 mm, vias 0 -> 1
- net COL3: track 66.1 -> 112.0 mm, vias 0 -> 1
- net COL4: track 65.2 -> 96.7 mm, vias 0 -> 2
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
Commit message: updating trace paths
Parts:
- moved F1 3.24 mm to (45.4, -103.1), turned to 180 degrees
- moved R1 0.65 mm to (35.6, -103.9)
- moved R2 0.28 mm to (39.2, -103.9)
- moved USB1 0.20 mm to (34.3, -122.9)
Connections:
- U1 pad 25: COL7 -> COL5
- U1 pad 27: COL5 -> COL7
- U1 pad 28: COL4 -> COL0
- U1 pad 29: COL3 -> COL1
- U1 pad 31: COL1 -> COL3
- U1 pad 32: COL0 -> COL4
Routing:
- net Net-(R1-Pad1): track 142.6 -> 118.8 mm, vias 2 -> 4
- net Net-(USB1-Pad6): track 0.00 -> 23.6 mm
- net COL4: track 96.7 -> 113.4 mm, vias 2 -> 3
- net ROW4: track 305.0 -> 319.6 mm, vias 2 -> 4
- net COL5: track 116.0 -> 128.8 mm
- net COL6: track 126.3 -> 136.9 mm
- net COL7: track 142.3 -> 150.3 mm
- net Net-(R2-Pad1): track 124.8 -> 117.0 mm, vias 2 -> 4
- net Net-(D52-Pad2): track 0.00 -> 7.03 mm
- net GND: track 269.7 -> 275.7 mm, vias 6 -> 5
- net ROW0: track 394.5 -> 389.8 mm, vias 8 -> 2
- net +5V: track 161.5 -> 157.6 mm, vias 6 -> 4
- net COL1: track 167.8 -> 171.5 mm
- net COL3: track 112.0 -> 109.0 mm, vias 1 -> 3
- net COL0: track 184.0 -> 186.7 mm
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- added copper zone on B.Cu, net GND

Commit message: fixes
Parts:
- moved SW1 1.85 mm to (133.8, -43.9)
- moved C3 1.85 mm to (124.2, -29.4)
- moved U1 1.85 mm to (116.6, -39.5)
- moved R4 1.85 mm to (107.6, -34.9)
- moved Y1 1.85 mm to (128.1, -39.2)
- moved C2 1.85 mm to (126.7, -29.4)
- moved C4 1.85 mm to (121.7, -29.4)
- moved C5 1.85 mm to (128.2, -34.8)
- moved C6 1.85 mm to (128.0, -43.7)
- moved C7 1.85 mm to (116.4, -48.6)
- moved R3 1.85 mm to (124.7, -46.0)
- moved C1 1.85 mm to (128.9, -29.4)
- moved MX27 0.13 mm to (144.6, -57.9)
Routing:
- net Net-(R2-Pad1): track 117.0 -> 120.9 mm
- net Net-(R1-Pad1): track 118.8 -> 121.5 mm
- net ROW3: track 322.8 -> 320.4 mm
- net COL13: track 262.9 -> 264.9 mm
- net COL9: track 192.7 -> 190.8 mm
- net ROW1: track 363.6 -> 365.1 mm
- net COL11: track 220.7 -> 219.5 mm
- net COL7: track 150.3 -> 149.0 mm
- net COL6: track 136.9 -> 135.7 mm
- net COL10: track 211.0 -> 209.9 mm
- net ROW4: track 319.6 -> 318.6 mm
- net GND: track 275.7 -> 276.7 mm
- net COL12: track 249.3 -> 248.4 mm
- net COL3: track 109.0 -> 108.2 mm
- net ROW0: track 389.8 -> 390.5 mm, vias 2 -> 4
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- removed copper zone on B.Cu, net GND

Commit message: FINAL
Parts:
- moved D62 1.84 mm to (307.3, -33.9)
- moved MX58 1.83 mm to (280.2, -34.1)
- moved MX62 1.78 mm to (299.2, -34.1)
- moved MX67 1.78 mm to (318.3, -34.1)
- moved D61 1.77 mm to (307.2, -53.1)
- moved MX61 1.76 mm to (299.2, -53.1)
- moved D67 1.72 mm to (326.3, -33.9)
- moved D58 1.59 mm to (288.1, -33.4)
- moved MX66 0.79 mm to (323.1, -57.9)
- moved MX63 0.78 mm to (323.1, -115.1)
- moved MX64 0.78 mm to (323.1, -96.1)
- moved MX65 0.78 mm to (323.1, -77.0)
- moved D64 0.76 mm to (331.0, -96.0)
- moved D65 0.64 mm to (330.8, -76.8)
- moved D66 0.64 mm to (330.8, -57.9)
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Routing:
- net COL14: track 283.8 -> 286.7 mm
- net COL13: track 264.9 -> 266.7 mm
- net ROW4: track 318.6 -> 320.4 mm
- net COL12: track 248.4 -> 250.0 mm
- net Net-(D67-Pad2): track 6.73 -> 7.68 mm
- net COL4: track 113.7 -> 112.9 mm
- net ROW3: track 320.4 -> 321.2 mm
- net ROW2: track 341.6 -> 342.1 mm
- added copper zone on B.Cu, net GND
Other:
- board outline added: 316.7 x 100 mm

Commit message: USB C JST addon
Parts:
- removed USB1: Molex-0548190589, random-keyboard-parts:Molex-0548190589
- added J2: Conn_01x04, random-keyboard-parts:JST-SR-4, B.Cu at (34.8, -120.7)
Routing:
- net Net-(USB1-Pad6): track 23.6 -> 0.00 mm
- net D+: track 15.5 -> 12.7 mm
- net D-: track 14.2 -> 11.6 mm
- net VCC: track 21.1 -> 18.6 mm

Commit message: Final keyboard file extraction
Parts:
- removed J2: Conn_01x04, random-keyboard-parts:JST-SR-4
- added R5: 5.1k, Resistor_SMD:R_0805_2012Metric_Pad1.15x1.40mm_HandSolder, B.Cu at (36.8, -114.2)
- added R6: 5.1k, Resistor_SMD:R_0805_2012Metric_Pad1.15x1.40mm_HandSolder, B.Cu at (33.0, -114.2)
- added USB1: Type-C_HRO-TYPE-C-31-M-12, Type-C:HRO-TYPE-C-31-M-12-HandSoldering, B.Cu at (34.7, -126.0)
- moved F1 6.35 mm to (44.3, -109.4), turned to 90 degrees
- moved R1 6.14 mm to (33.0, -109.5)
- moved R2 6.10 mm to (36.8, -109.5)
- moved D1 3.18 mm to (28.6, -110.2)
Routing:
- net GND: track 277.2 -> 299.0 mm
- net Net-(R2-Pad1): track 120.9 -> 127.5 mm
- net Net-(R1-Pad1): track 121.5 -> 127.7 mm
- net +5V: track 157.4 -> 162.3 mm
- net ROW0: track 390.7 -> 394.3 mm
- net Net-(R6-Pad1): track 0.00 -> 2.83 mm
- net Net-(R5-Pad1): track 0.00 -> 2.81 mm
- net D+: track 12.7 -> 14.9 mm
- net VCC: track 18.6 -> 20.5 mm, vias 2 -> 0
- net Net-(D1-Pad2): track 9.64 -> 7.99 mm
- net D-: track 11.6 -> 10.7 mm
- added copper zone on F.Cu, net GND
